Commit message: Validate CR5 mount + teleop on real hardware config, add livestream support
CR5 validation: mount the real CR5 URDF instead of the temporary Franka
override, fixing four bugs surfaced along the way -- zero URDF velocity
limits, an overlapping collision sphere, an incomplete self-collision-ignore
list, and a singular all-zero retract_config (replaced with a bent-elbow
pose). Recomputed teleop_target's FK-derived pose to match. Pinned
TORCH_CUDA_ARCH_LIST for the L4 GPU this was validated against.

build_scene.py:
- Add --livestream, reusing the isaacsim.exp.full.streaming.kit experience
  isaac-sim.streaming.sh already uses, with hide_ui=False so the full UI
  streams (SimulationApp's own headless=True default hides it otherwise).
  Default (no flags) now explicitly opens isaacsim.exp.full.kit for the
  local GUI case, matching mefron.py's convention. Add the
  preload_real_packaging() guard this full-experience path requires.
- Fix run_teleop_loop() to rebuild robot/idx_list/articulation_controller
  on every fresh Play, not just once -- matches mefron_lib/teleop.py's
  already-correct pattern (see CLAUDE.md's Stop/Play rebuild gotcha).
- Gate cmd_plan waypoint application on real elapsed time
  (result.interpolation_dt) instead of one waypoint per simulation_app
  update() call, so playback speed doesn't outrun the planned trajectory.
- Remove the temporary _SKIP_ROBOT_FOR_DRAGDROP_TEST detour.

Co-Authored-By: Claude Sonnet 5 <noreply@anthropic.com>

File: robots/cr5/urdf/cr5_robot.urdf (robot description, URDF)
Before this commit: robot cr5_robot, 8 links, 7 joints
Joints:
- joint joint1: limit lower=-3.14 upper=3.14 effort=0 velocity=0 -> lower=-3.14 upper=3.14 effort=0 velocity=3.14
- joint joint2: limit lower=-3.14 upper=3.14 effort=0 velocity=0 -> lower=-3.14 upper=3.14 effort=0 velocity=3.14
- joint joint3: limit lower=-2.86 upper=2.86 effort=0 velocity=0 -> lower=-2.86 upper=2.86 effort=0 velocity=3.14
- joint joint4: limit lower=-3.14 upper=3.14 effort=0 velocity=0 -> lower=-3.14 upper=3.14 effort=0 velocity=3.14
- joint joint5: limit lower=-3.14 upper=3.14 effort=0 velocity=0 -> lower=-3.14 upper=3.14 effort=0 velocity=3.14
- joint joint6: limit lower=-6.28 upper=6.28 effort=0 velocity=0 -> lower=-6.28 upper=6.28 effort=0 velocity=3.14
